Commit message: Revert "Rainbow: wrist-camera and ZED collision spheres (n_spheres 196 -> 199)"
This reverts commit 897b5967384670e2bbd936a145ce874232d53da7.

File: resources/rainbow/rainbow_spherized.urdf (robot description, URDF)
Before this commit: robot RB_Y1_V1.0.1, 42 links, 41 joints
Links:
- removed link link_left_arm_camera
- removed link link_right_arm_camera
- link rby1_camera_mount: geometry visual mesh filename=./meshes/rby1_camera_mount_realsense.obj
Joints:
- removed joint left_arm_camera_mount
- removed joint right_arm_camera_mount
