Commit message: Rainbow: 23-DOF dual-arm model + left-attachment twin vamp.rainbowl
rainbow.hh regenerated with torso_0..5 and left_arm_0..6 opened up
(x, y, theta, torso 6, left 7, right 7; head stays baked). New module
rainbowl: identical DOF/spheres, attachment frame grasp_frame_left (a
model bakes one attachment frame; per-hand attachment = per-hand module).
Fixed grasp_joint_left z offset sign (+0.13 -> -0.13, matching
rainbow_seiji.urdf; 260mm left-EE error while unused).

Co-Authored-By: Claude Fable 5 <noreply@anthropic.com>

File: resources/rainbow/rainbow_spherized.urdf (robot description, URDF)
Before this commit: robot RB_Y1_V1.0.1, 40 links, 39 joints
Links:
- link base: geometry collision sphere radius=0.08; collision sphere radius=0.08
- link link_torso_0: geometry collision sphere radius=0.13; collision sphere radius=0.13
- link link_torso_1: geometry collision sphere radius=0.11; collision sphere radius=0.11
- link link_torso_2: geometry collision sphere radius=0.11; collision sphere radius=0.11
- link link_torso_4: geometry collision sphere radius=0.12; collision sphere radius=0.15
Joints:
- joint grasp_joint_left: origin xyz=0 0 0.13 rpy=0 0 -1.57079632679 -> xyz=0 0 -0.13 rpy=0 0 -1.57079632679
- joint left_arm_0: type fixed -> revolute
- joint left_arm_1: type fixed -> revolute
- joint left_arm_2: type fixed -> revolute
- joint left_arm_3: type fixed -> revolute
- joint left_arm_4: type fixed -> revolute
- joint left_arm_5: type fixed -> revolute
- joint left_arm_6: type fixed -> revolute
- joint torso_0: axis (none) -> 1 0 0; limit (none) -> lower=-0.261799388 upper=0.261799388 effort=270.0 velocity=2.09439510; type fixed -> revolute
- joint torso_1: axis (none) -> 0 1 0; limit (none) -> lower=-0.523598776 upper=1.570796327 effort=270.0 velocity=2.09439510; origin xyz=0.0 0.0 0.0 rpy=0.0 0.523599 0.0 -> xyz=0.0 0.0 0.0 rpy=0.0 0.0 0.0; type fixed -> revolute
- joint torso_2: axis (none) -> 0 1 0; limit (none) -> lower=-2.617993878 upper=1.570796327 effort=270.0 velocity=2.09439510; origin xyz=0.0 0.0 0.350 rpy=0.0 -1.0472 0.0 -> xyz=0.0 0.0 0.350 rpy=0.0 0.0 0.0; type fixed -> revolute
- joint torso_3: axis (none) -> 0 1 0; limit (none) -> lower=-0.785398163 upper=1.570796327 effort=120.0 velocity=3.141592654; origin xyz=0.0 0.0 0.350 rpy=0.0 0.785398 0.0 -> xyz=0.0 0.0 0.350 rpy=0.0 0.0 0.0; type fixed -> revolute
- joint torso_4: axis (none) -> 1 0 0; limit (none) -> lower=-0.523598776 upper=0.523598776 effort=120.0 velocity=3.141592654; type fixed -> revolute
- joint torso_5: axis (none) -> 0 0 1; limit (none) -> lower=-2.35619449 upper=2.35619449 effort=120.0 velocity=3.141592654; type fixed -> revolute

Commit message: Rainbow: rebound 18 joints to match the Drake rby1 model
Joint limits are compiled into the generated headers in four places:
the s_a/s_m/d_m arrays and the two unrolled per-index scale/descale
blocks. Nothing else in these files is limit-derived — the sphere FK
is independent — so a limits-only change needs no cricket regen.

Verified after rebuild: lower_bounds()/upper_bounds() match
rainbow_seiji.urdf with 0 mismatches, d_m == 1/s_m, and both unrolled
blocks agree with the arrays. Base joints (x, y, theta) untouched.
n_spheres unchanged at 196.

Co-Authored-By: Claude Opus 4.8 <noreply@anthropic.com>

File: resources/rainbow/rainbow_spherized.urdf (robot description, URDF)
Before this commit: robot RB_Y1_V1.0.1, 40 links, 39 joints
Joints:
- joint head_1: limit lower=-0.35 upper=0.785 effort=1000 velocity=3.14 -> lower=-0.35 upper=1.57 effort=1000 velocity=3.14
- joint left_arm_0: limit lower=-3.141592654 upper=3.141592654 effort=70.0 velocity=3.141592654 -> lower=-2.35619449 upper=2.35619449 effort=70.0 velocity=3.141592654
- joint left_arm_1: limit lower=-0.017453293 upper=3.141592654 effort=70.0 velocity=3.141592654 -> lower=-0.05 upper=3.141592654 effort=70.0 velocity=3.141592654
- joint left_arm_2: limit lower=-3.141592654 upper=3.141592654 effort=70.0 velocity=3.141592654 -> lower=-2.09439510 upper=2.09439510 effort=70.0 velocity=3.141592654
- joint left_arm_3: limit lower=-2.617993878 upper=0.017453293 effort=40.0 velocity=3.141592654 -> lower=-2.617993878 upper=0.01 effort=40.0 velocity=3.141592654
- joint left_arm_4: limit lower=-3.141592654 upper=3.141592654 effort=10.0 velocity=6.283185308 -> lower=-3.0 upper=3.0 effort=10.0 velocity=6.283185308
- joint left_arm_5: limit lower=-1.570796327 upper=1.919862177 effort=10.0 velocity=6.283185308 -> lower=-1.74532925 upper=2.00712864 effort=10.0 velocity=6.283185308
- joint left_arm_6: limit lower=-2.705260340 upper=2.705260340 effort=8.0 velocity=2.094395102 -> lower=-2.75 upper=2.75 effort=8.0 velocity=2.094395102
- joint right_arm_0: limit lower=-3.141592654 upper=3.141592654 effort=70.0 velocity=3.141592654 -> lower=-2.35619449 upper=2.35619449 effort=70.0 velocity=3.141592654
- joint right_arm_1: limit lower=-3.141592654 upper=0.017453293 effort=70.0 velocity=3.141592654 -> lower=-3.141592654 upper=0.05 effort=70.0 velocity=3.141592654
- joint right_arm_2: limit lower=-3.141592654 upper=3.141592654 effort=70.0 velocity=3.141592654 -> lower=-2.09439510 upper=2.09439510 effort=70.0 velocity=3.141592654
- joint right_arm_3: limit lower=-2.617993878 upper=0.017453293 effort=40.0 velocity=3.141592654 -> lower=-2.617993878 upper=0.01 effort=40.0 velocity=3.141592654
- joint right_arm_4: limit lower=-3.141592654 upper=3.141592654 effort=10.0 velocity=6.283185308 -> lower=-3.0 upper=3.0 effort=10.0 velocity=6.283185308
- joint right_arm_5: limit lower=-1.570796327 upper=1.919862177 effort=10.0 velocity=6.283185308 -> lower=-1.74532925 upper=2.00712864 effort=10.0 velocity=6.283185308
- joint right_arm_6: limit lower=-2.705260340 upper=2.705260340 effort=8.0 velocity=2.094395102 -> lower=-2.75 upper=2.75 effort=8.0 velocity=2.094395102
- joint torso_0: limit lower=-0.261799388 upper=0.261799388 effort=270.0 velocity=2.09439510 -> lower=-0.34906585 upper=0.34906585 effort=270.0 velocity=2.09439510
- joint torso_1: limit lower=-0.523598776 upper=1.570796327 effort=270.0 velocity=2.09439510 -> lower=-1.04719755 upper=1.52173048 effort=270.0 velocity=2.09439510
- joint torso_2: limit lower=-2.617993878 upper=1.570796327 effort=270.0 velocity=2.09439510 -> lower=-2.478367 upper=1.570796327 effort=270.0 velocity=2.09439510
- joint torso_5: limit lower=-2.35619449 upper=2.35619449 effort=120.0 velocity=3.141592654 -> lower=-1.57079633 upper=1.57079633 effort=120.0 velocity=3.141592654

Commit message: Rainbow: wrist-camera and ZED collision spheres (n_spheres 196 -> 199)
Regenerated from cricket with the new geometry. Sphere sizing note: the wrist
camera uses the MESH's minimal enclosing sphere (r=0.04668 at the mesh's true
centre), NOT the bounding sphere of the declared box (r=0.05353). The mesh sits
1.7 cm off-centre inside its box, so the box-derived sphere is both 13% too big
and displaced OUTBOARD -- the direction that costs clearance. Multi-sphere covers
are worse here: minimising centre+radius over a box is monotone in the centre, so
the single centred sphere is the shallowest cover, and the binding dimension is
vertical (fingertip clearance under an overhang), not lateral.

srdf: the three new links are APPENDED to the original file byte-for-byte, each
inheriting the live-disable set of the link it is bolted to (rby1_camera_mount <-
link_head_2, link_{r,l}_arm_camera <- FT_sensor_{R,L}), so the deliberately-enabled
self-collision pairs survive. 561 -> 621 entries.

KNOWN LIMITATION: this vamp model is 23-DOF with no head joints, so the ZED sphere
on rby1_camera_mount is frozen at head-zero and cannot track head pose -- off by
6.8 cm at the default head conf, 18.6 cm at full tilt. It cannot matter in a
tabletop scene (it sits ~1.4 m up) but should be revisited.

Co-Authored-By: Claude Opus 4.8 <noreply@anthropic.com>

File: resources/rainbow/rainbow_spherized.urdf (robot description, URDF)
Before this commit: robot RB_Y1_V1.0.1, 40 links, 39 joints
Links:
- added link link_left_arm_camera; collision sphere radius=0.04668
- added link link_right_arm_camera; collision sphere radius=0.04668
- link rby1_camera_mount: geometry collision sphere radius=0.095; visual mesh filename=./meshes/rby1_camera_mount_realsense.obj
Joints:
- added joint left_arm_camera_mount: type fixed, parent FT_sensor_L, child link_left_arm_camera, origin xyz=0 0 0 rpy=0 0 0
- added joint right_arm_camera_mount: type fixed, parent FT_sensor_R, child link_right_arm_camera, origin xyz=0 0 0 rpy=0 0 0

Commit message: Rainbow: split into vamp.rainbow (197) and vamp.rainbowcam (199)
Two selectable collision models sharing all kinematics; the wrist cameras are
the only difference (ZED head sphere + lidar on both):
  * rainbow.hh / rainbowl.hh       -- 197 spheres (196 + ZED)
  * rainbowcam.hh / rainbowcaml.hh -- 199 spheres (+2 wrist-camera spheres)

Both parallel build lists updated: VAMP_ROBOT_MODULES += rainbowcam;rainbowcaml
and VAMP_ROBOT_STRUCTS += RainbowCam;RainbowCaml (they are ZIP'd -- a mismatch
fails the build). Verified after rebuild: rainbowcam's shared 197 spheres are
byte-identical to rainbow's at a probe conf (max distance 0.0), the 2 extra
spheres sit at the wrist, and both models' default posture is collision-free.

Co-Authored-By: Claude Opus 4.8 <noreply@anthropic.com>

File: resources/rainbow/rainbow_spherized.urdf (robot description, URDF)
Before this commit: robot RB_Y1_V1.0.1, 40 links, 39 joints
Links:
- link rby1_camera_mount: geometry collision sphere radius=0.095; visual mesh filename=./meshes/rby1_camera_mount_realsense.obj
